File: PCB/MacroCAD.kicad_pcb (KiCad board)
At the start: 2 copper layers, 72 x 95.5 mm, 28 parts, among them J1 Conn_01x04, SW1 SW_Push, SW10 SW_Push, SW11 SW_Push, SW12 SW_Push, SW2 SW_Push, SW3 SW_Push, SW4 SW_Push, SW5 SW_Push, SW6 SW_Push, SW7 SW_Push, SW8 SW_Push, SW9 SW_Push, U1 MOUDLE-SEEEDUINO-XIAO

Commit message: PCB's final toutch
Parts:
- J1: value Conn_01x04 -> OLED SCREEN
Connections:
- net Net-(D1-K) renamed D0
- net Net-(D10-K) renamed D1
- net Net-(D11-K) renamed D2
- net Net-(D12-K) renamed D3
- net Net-(J1-Pin_3) renamed D5
- net Net-(J1-Pin_4) renamed D4
- net Net-(U1-PA5_A9_D9_MISO) renamed D9
- net Net-(U1-PA6_A10_D10_MOSI) renamed D10
- net Net-(U1-PA7_A8_D8_SCK) renamed D8
